File: kicad/mce-adapter.sch (KiCad schematic (older format))
At the start: 19 parts, among them J123 Conn_02x03_Odd_Even, J4 Conn_01x03_Male, SW1 SW_DIP_x03, U1 GAL16V8

Commit message: Fixed GAL name
Parts:
- R7: value 75 -> 100
- U1: value GAL16V8 -> GAL16V8B
Changed lines of the file:
@@
 P 4100 2650
 F 0 "U1" H 4100 2800 50  0000 C CNN
-F 1 "GAL16V8" H 4100 2700 50  0000 C CNN
+F 1 "GAL16V8B" H 4100 2700 50  0000 C CNN
 F 2 "Package_DIP:DIP-20_W7.62mm_Socket" H 4100 2650 50  0001 C CNN
 F 3 "" H 4100 2650 50  0001 C CNN
@@
 P 4900 2150
 F 0 "R7" V 4850 2000 50  0000 C CNN
-F 1 "75" V 4900 2150 50  0000 C CNN
+F 1 "100" V 4900 2150 50  0000 C CNN
 F 2 "Resistor_THT:R_Axial_DIN0204_L3.6mm_D1.6mm_P7.62mm_Horizontal" V 4830 2150 50  0001 C CNN
 F 3 "~" H 4900 2150 50  0001 C CNN
